File: DBA/DBA.kicad_sch (KiCad schematic)
At the start: 11 parts, among them J1 USB_B_Micro, J4 Conn_01x01_Male, J5 Conn_01x01_Male, U1 ESP32_NodeMCU_v1.1, U2 MCP1700-3302E_TO92

Commit message: first circular version{
Parts:
- BT1: footprint Battery:BatteryHolder_Keystone_1042_1x18650 -> Battery:Battery_Custom
Changed lines of the file:
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@@
     (property "Reference" "BT1" (id 0) (at 105.918 52.07 90))
     (property "Value" "Battery_Cell" (id 1) (at 105.918 54.61 90))
-    (property "Footprint" "Battery:BatteryHolder_Keystone_1042_1x18650" (id 2) (at 106.426 59.69 90)
+    (property "Footprint" "Battery:Battery_Custom" (id 2) (at 106.426 59.69 90)
       (effects (font (size 1.27 1.27)) hide)
     )
@@
     )
     (path "/c81e662e-4d27-4fc0-ab76-275983e79520"
-      (reference "BT1") (unit 1) (value "Battery_Cell") (footprint "Battery:BatteryHolder_Keystone_1042_1x18650")
+      (reference "BT1") (unit 1) (value "Battery_Cell") (footprint "Battery:Battery_Custom")
     )
     (path "/d441a738-aa4d-42f2-86bb-fdcfdbf0c359"
